Commit message: Editing stls

File: src/clam_description/urdf/clam.xacro (robot description, xacro)
@@ -343,4 +343,10 @@
       <material name="Orange" />
     </visual>
+    <collision>
+      <origin xyz="0 0 0" rpy="0 0 0" />
+      <geometry>
+        <mesh filename="package://clam_description/stl/gripper_grip_link_simple.STL" scale="1 1 1" />
+      </geometry>
+    </collision>
   </link>
   <gazebo reference="gripper_roll_link">
