Commit message: Testing arm reach on workspace

File: src/clam_description/urdf/clam.urdf (robot description, URDF)
Before this commit: robot clam, 15 links, 14 joints
Links:
- removed link gripper_link
- added link camera_calibration_link; visual sphere radius=.001
- added link tabletop_link; visual mesh filename=package://clam_description/stl/tabletop.STL scale=1 1 1
Joints:
- removed joint gripper_link_joint
- added joint camera_calibration_link_joint: type fixed, parent gripper_roll_link, child camera_calibration_link, origin xyz=0.1795 0.002 0 rpy=0 0 0
- added joint tabletop_joint: type fixed, parent base_link, child tabletop_link, origin xyz=0 0 0 rpy=0 0 0

File: src/clam_description/urdf/clam.xacro (robot description, xacro)
@@ -312,5 +312,5 @@
   </link>
   <!-- TABLETOP MODEL -->
-  <!--joint name="tabletop_joint" type="fixed">
+  <joint name="tabletop_joint" type="fixed">
     <origin xyz="0 0 0" rpy="0 0 0" />
     <parent link="base_link"/>
@@ -325,13 +325,12 @@
       <material name="Brown" />
     </visual>
-  </link-->
-  <!-- FAKE CAMERA CALIBRATION POINT AT GRIPPER TIP  -->
-  <joint name="gripper_link_joint" type="fixed">
-    <!--origin xyz="0.012 -0.11 0.020" rpy="0 0 0" /-->
-    <origin xyz="0.1795 0 0" rpy="0 0 0" />
-    <parent link="gripper_roll_link"/>
-    <child link="gripper_link" />
-  </joint>
-  <link name="gripper_link" >
+  </link>
+  <!-- FAKE CAMERA CALIBRATION POINT AT GRIPPER TIP -->
+  <joint name="camera_calibration_link_joint" type="fixed">
+    <origin xyz="0.1795 0.002 0" rpy="0 0 0" />
+    <parent link="gripper_roll_link"/>
+    <child link="camera_calibration_link" />
+  </joint>
+  <link name="camera_calibration_link" >
     <visual>
       <origin xyz="0 0 0" rpy="0 0 0" />

Commit message: Renamed links in URDF and SRDF

File: src/clam_description/urdf/clam.urdf (robot description, URDF)
Before this commit: robot clam, 16 links, 15 joints
Links:
- removed link camera_calibration_link
- added link gripper_fake_tip_link; visual sphere radius=.001
Joints:
- removed joint camera_calibration_link_joint
- removed joint l_gripper_fwd_link_joint
- removed joint r_gripper_aft_link_joint
- removed joint r_gripper_fwd_link_joint
- added joint gripper_fake_tip_joint: type fixed, parent gripper_roll_link, child gripper_fake_tip_link, origin xyz=0.1795 0.002 0 rpy=0 0 0
- added joint l_gripper_fwd_joint: type revolute, parent gripper_roll_link, child l_gripper_fwd_link, origin xyz=0.05 0.008 0.007 rpy=3.2672536 1.570795 3.74512434556, axis 1 0 0, limit lower=0 upper=1.57 effort=300 velocity=1, mimic joint=l_gripper_aft_joint multiplier=1.0 offset=0
- added joint r_gripper_aft_joint: type revolute, parent gripper_roll_link, child r_gripper_aft_link, origin xyz=0.026 -0.011  0 rpy=4.22543855 1.570795 0.603534345556, axis 1 0 0, limit lower=-3.14 upper=3.14 effort=300 velocity=1, mimic joint=l_gripper_aft_joint multiplier=-1.0 offset=0.0
- added joint r_gripper_fwd_joint: type revolute, parent gripper_roll_link, child r_gripper_fwd_link, origin xyz=0.05 -0.0014 0.007 rpy=3.0159264 1.570795 2.53805565444, axis 1 0 0, limit lower=-1.57 upper=0 effort=300 velocity=1, mimic joint=l_gripper_aft_joint multiplier=-1.0 offset=0

File: src/clam_description/urdf/clam.xacro (robot description, xacro)
@@ -216,5 +216,5 @@
     </visual>
   </link>
-  <joint name="r_gripper_aft_link_joint" type="revolute">
+  <joint name="r_gripper_aft_joint" type="revolute">
     <parent link="gripper_roll_link"/>
     <child link="r_gripper_aft_link"/>
@@ -235,5 +235,5 @@
     </visual>
   </link>
-  <joint name="l_gripper_fwd_link_joint" type="revolute">
+  <joint name="l_gripper_fwd_joint" type="revolute">
     <parent link="gripper_roll_link"/>
     <child link="l_gripper_fwd_link"/>
@@ -254,5 +254,5 @@
     </visual>
   </link>
-  <joint name="r_gripper_fwd_link_joint" type="revolute">
+  <joint name="r_gripper_fwd_joint" type="revolute">
     <parent link="gripper_roll_link"/>
     <child link="r_gripper_fwd_link"/>
@@ -327,10 +327,10 @@
   </link>
   <!-- FAKE CAMERA CALIBRATION POINT AT GRIPPER TIP -->
-  <joint name="camera_calibration_link_joint" type="fixed">
+  <joint name="gripper_fake_tip_joint" type="fixed">
     <origin xyz="0.1795 0.002 0" rpy="0 0 0" />
     <parent link="gripper_roll_link"/>
-    <child link="camera_calibration_link" />
-  </joint>
-  <link name="camera_calibration_link" >
+    <child link="gripper_fake_tip_link" />
+  </joint>
+  <link name="gripper_fake_tip_link" >
     <visual>
       <origin xyz="0 0 0" rpy="0 0 0" />

Commit message: Renamed stuff in URDF

File: src/clam_description/urdf/clam.urdf (robot description, URDF)
Before this commit: robot clam, 16 links, 15 joints
Links:
- removed link l_gripper_pincher
- removed link r_gripper_pincher
- added link l_gripper_pincher_link; visual mesh filename=package://clam_description/stl/l_gripper_pincher.STL scale=1 1 1
- added link r_gripper_pincher_link; visual mesh filename=package://clam_description/stl/r_gripper_pincher.STL scale=1 1 1
Joints:
- joint l_gripper_aft_pincher_joint: child l_gripper_pincher -> l_gripper_pincher_link
- joint r_gripper_aft_pincher_joint: child r_gripper_pincher -> r_gripper_pincher_link

File: src/clam_description/urdf/clam.xacro (robot description, xacro)
@@ -275,5 +275,5 @@
   <joint name="l_gripper_aft_pincher_joint" type="continuous">
     <parent link="l_gripper_aft_link"/>
-    <child link="l_gripper_pincher"/>
+    <child link="l_gripper_pincher_link"/>
     <origin xyz="-0.0032 0 -0.0508" rpy="${203.27*M_PI/180-.3150*M_PI} 0 0" />
     <axis xyz="1 0 0" />
@@ -283,5 +283,5 @@
   </joint>
   <!-- LEFT GRIPPER PINCHER -->
-  <link name="l_gripper_pincher">
+  <link name="l_gripper_pincher_link">
     <visual>
       <origin xyz="0 0 0" rpy="0 0 ${M_PI}" />
@@ -294,5 +294,5 @@
   <joint name="r_gripper_aft_pincher_joint" type="revolute">
     <parent link="r_gripper_aft_link"/>
-    <child link="r_gripper_pincher"/>
+    <child link="r_gripper_pincher_link"/>
     <origin xyz="0 0 -0.0508" rpy="${23.27*M_PI/180-.3150*M_PI} ${M_PI} 0" />
     <axis xyz="1 0 0" />
@@ -302,5 +302,5 @@
   </joint>
   <!-- RIGHT GRIPPER PINCHER -->
-  <link name="r_gripper_pincher">
+  <link name="r_gripper_pincher_link">
     <visual>
       <origin xyz="0 0 0" rpy="0 0 ${M_PI}" />

Commit message: Created ClamArm gazebo model

File: src/clam_description/urdf/clam.urdf (robot description, URDF)
Before this commit: robot clam, 16 links, 15 joints
Links:
- link base_link: mass None -> 1.0
- link elbow_pitch_link: mass None -> 1.0
- link elbow_roll_link: mass None -> 1.0
- link gripper_fake_tip_link: mass None -> 1.0
- link gripper_roll_link: mass None -> 1.0
- link l_gripper_aft_link: mass None -> 1.0
- link l_gripper_fwd_link: mass None -> 1.0
- link l_gripper_pincher_link: mass None -> 1.0
- link r_gripper_aft_link: mass None -> 1.0
- link r_gripper_fwd_link: mass None -> 1.0
- link r_gripper_pincher_link: mass None -> 1.0
- link shoulder_pan_link: mass None -> 1.0
- link shoulder_pitch_link: mass None -> 1.0
- link tabletop_link: mass None -> 1.0
- link wrist_pitch_link: mass None -> 1.0
- link wrist_roll_link: mass None -> 1.0

File: src/clam_description/urdf/clam.xacro (robot description, xacro)
@@ -2,5 +2,5 @@
 <!-- Robot Description format of CLAM arm
 Dave Coleman - davetcoleman@gmail.com
-1/10/2012
+12/20/2012
 Documentation:
 URDF
@@ -10,4 +10,6 @@
 XARCO - Macro Language
 http://www.ros.org/wiki/xacro
+Gazebo Modeling
+http://www.ros.org/wiki/simulator_gazebo/Tutorials/SpawningObjectInSimulation
 -->
 <robot name="clam"
@@ -20,10 +22,87 @@
   <property name="M_SCALE" value="0.001 0.001 0.001"/>
   <property name="M_PI" value="3.14159"/>
+  <!-- Add a Gazebo plugin controller -->
+  <gazebo>
+    <controller:gazebo_ros_actuator_array
+        name="actuator_array_controller"
+        plugin="libgazebo_ros_actuator_array.so">
+      <alwaysOn>true</alwaysOn>
+      <updateRate>50.0</updateRate>
+      <robotParam>robot_description</robotParam>
+      <joint>
+        <name>joint1</name>
+        <home>0.0</home>
+        <p>10.0</p>
+        <i>0.0</i>
+        <d>0.0</d>
+        <iClamp>0.0</iClamp>
+      </joint>
+      <joint>
+        <name>joint2</name>
+        <home>2.094395102</home>
+        <p>10.0</p>
+        <i>0.0</i>
+        <d>0.0</d>
+        <iClamp>0.0</iClamp>
+      </joint>
+      <joint>
+        <name>joint3</name>
+        <home>1.483529864</home>
+        <p>10.0</p>
+        <i>0.0</i>
+        <d>0.0</d>
+        <iClamp>0.0</iClamp>
+      </joint>
+      <joint>
+        <name>joint4</name>
+        <home>0.0</home>
+        <p>10.0</p>
+        <i>0.0</i>
+        <d>0.0</d>
+        <iClamp>0.0</iClamp>
+      </joint>
+    </controller:gazebo_ros_actuator_array>
+  </gazebo>
+  <!-- TABLETOP LINK -->
+  <joint name="tabletop_joint" type="fixed">
+    <origin xyz="0 0 0" rpy="0 0 0" />
+    <parent link="base_link"/>
+    <child link="tabletop_link"/>
+  </joint>
+  <link name="tabletop_link">
+    <inertial>
+      <origin xyz=" 0 0 -0.017"/>
+      <mass value="100.0" />
+      <inertia  ixx="1.0" ixy="0.0"  ixz="0.0"  iyy="100.0"  iyz="0.0"  izz="1.0" />
+    </inertial>
+    <visual>
+      <origin xyz=" 0 0 -0.017"  rpy="${.5*M_PI} 0 ${.5*M_PI}"/>
+      <geometry>
+        <mesh filename="package://clam_description/stl/tabletop.STL" scale="1 1 1" />
+      </geometry>
+      <material name="Brown" />
+    </visual>
+    <collision>
+      <origin xyz=" 0 0 -0.017"  rpy="${.5*M_PI} 0 ${.5*M_PI}"/>
+      <geometry>
+        <mesh filename="package://clam_description/stl/tabletop.STL" scale="1 1 1" />
+      </geometry>
+      </collision>>
+  </link>
+  <gazebo reference="tabletop_link">
+    <material>Gazebo/WoodFloor</material>
+    <turnGravityOff>false</turnGravityOff>
+  </gazebo>
   <!-- BASE LINK -->
   <link name="base_link">
+    <inertial>
+      <origin xyz="0 0 0" />
+      <mass value="1.0" />
+      <inertia  ixx="1.0" ixy="0.0"  ixz="0.0"  iyy="100.0"  iyz="0.0"  izz="1.0" />
+    </inertial>
     <visual>
       <origin xyz="0 0 0" rpy="${M_PI/2} 0 0" /> <!-- rotate PI/2 -->
       <geometry>
-	<mesh filename="package://clam_description/stl/base_link.STL" scale="${M_SCALE}" />
+        <mesh filename="package://clam_description/stl/base_link.STL" scale="${M_SCALE}" />
       </geometry>
       <material name="Grey" />
@@ -32,8 +111,12 @@
       <origin xyz="0 0 0" rpy="${M_PI/2} 0 0" /> <!-- rotate PI/2 -->
       <geometry>
-	<mesh filename="package://clam_description/stl/base_link_simple.STL" scale="${M_SCALE}" />
+        <mesh filename="package://clam_description/stl/base_link_simple.STL" scale="${M_SCALE}" />
       </geometry>
       </collision>>
   </link>
+  <gazebo reference="base_link">
+    <material>Gazebo/Blue</material>
+    <turnGravityOff>false</turnGravityOff>
+  </gazebo>
   <joint name="shoulder_pan_joint" type="revolute">
     <parent link="base_link"/>
@@ -44,10 +127,21 @@
     <dynamics damping="50" friction="1"/>
   </joint>
+  <transmission name="shoulder_pan_controller" type="pr2_mechanism_model/SimpleTransmission">
+    <actuator name="shoulder_pan_actuator" />
+    <joint name="shoulder_pan_joint" />
+    <mechanicalReduction>1</mechanicalReduction>
+    <motorTorqueConstant>1</motorTorqueConstant>
+  </transmission>
   <!-- SHOULDER PAN LINK -->
   <link name="shoulder_pan_link" >
+    <inertial>
+      <origin xyz="0 0 0" />
+      <mass value="1.0" />
+      <inertia  ixx="1.0" ixy="0.0"  ixz="0.0"  iyy="100.0"  iyz="0.0"  izz="1.0" />
+    </inertial>
     <visual>
       <origin xyz="0 0 0" rpy="0 0 ${M_PI/2}" />
       <geometry>
-	<mesh filename="package://clam_description/stl/shoulder_pan_link.STL" scale="${M_SCALE}" />
+        <mesh filename="package://clam_description/stl/shoulder_pan_link.STL" scale="${M_SCALE}" />
       </geometry>
       <material name="Orange" />
@@ -56,8 +150,12 @@
       <origin xyz="0 0 0" rpy="0 0 ${M_PI/2}" />
       <geometry>
-	<mesh filename="package://clam_description/stl/shoulder_pan_link_simple.STL" scale="${M_SCALE}" />
+        <mesh filename="package://clam_description/stl/shoulder_pan_link_simple.STL" scale="${M_SCALE}" />
       </geometry>
     </collision>
   </link>
+  <gazebo reference="shoulder_pan_link">
+    <material>Gazebo/Blue</material>
+    <turnGravityOff>false</turnGravityOff>
+  </gazebo>
   <joint name="shoulder_pitch_joint" type="revolute">
     <parent link="shoulder_pan_link"/>
@@ -70,8 +168,13 @@
   <!-- SHOULDER PITCH LINK -->
   <link name="shoulder_pitch_link" >
+    <inertial>
+      <origin xyz="-0.002 0 -0.000"  />
+      <mass value="1.0" />
+      <inertia  ixx="1.0" ixy="0.0"  ixz="0.0"  iyy="100.0"  iyz="0.0"  izz="1.0" />
+    </inertial>
     <visual>
       <origin xyz="-0.002 0 -0.000" rpy="${M_PI/2} ${M_PI} ${M_PI/2}" />
       <geometry>
-	<mesh filename="package://clam_description/stl/shoulder_pitch_link.STL" scale="${M_SCALE}" />
+        <mesh filename="package://clam_description/stl/shoulder_pitch_link.STL" scale="${M_SCALE}" />
       </geometry>
       <material name="Grey" />
@@ -80,8 +183,12 @@
       <origin xyz="-0.002 0 -0.000" rpy="${M_PI/2} ${M_PI} ${M_PI/2}" />
       <geometry>
-	<mesh filename="package://clam_description/stl/shoulder_pitch_link_simple.STL" scale="${M_SCALE}" />
+        <mesh filename="package://clam_description/stl/shoulder_pitch_link_simple.STL" scale="${M_SCALE}" />
       </geometry>
     </collision>
   </link>
+  <gazebo reference="shoulder_pitch_link">
+    <material>Gazebo/Blue</material>
+    <turnGravityOff>false</turnGravityOff>
+  </gazebo>
   <joint name="elbow_roll_joint" type="revolute">
     <parent link="shoulder_pitch_link"/>
@@ -94,8 +201,13 @@
   <!-- ELBOW ROLL LINK -->
   <link name="elbow_roll_link" >
+    <inertial>
+      <origin xyz="-0.035 0.0 0.0"  />
+      <mass value="1.0" />
+      <inertia  ixx="1.0" ixy="0.0"  ixz="0.0"  iyy="100.0"  iyz="0.0"  izz="1.0" />
+    </inertial>
     <visual>
       <origin xyz="-0.035 0.0 0.0" rpy="${M_PI} ${M_PI/2} ${M_PI/2}" />
       <geometry>
-	<mesh filename="package://clam_description/stl/elbow_roll_link.STL" scale="${M_SCALE}" />
+        <mesh filename="package://clam_description/stl/elbow_roll_link.STL" scale="${M_SCALE}" />
       </geometry>
       <material name="Black" />
@@ -104,8 +216,12 @@
       <origin xyz="-0.035 0.0 0.0" rpy="${M_PI} ${M_PI/2} ${M_PI/2}" />
       <geometry>
-	<mesh filename="package://clam_description/stl/elbow_roll_link_simple.STL" scale="${M_SCALE}" />
+        <mesh filename="package://clam_description/stl/elbow_roll_link_simple.STL" scale="${M_SCALE}" />
       </geometry>
     </collision>
   </link>
+  <gazebo reference="elbow_roll_link">
+    <material>Gazebo/Blue</material>
+    <turnGravityOff>false</turnGravityOff>
+  </gazebo>
   <joint name="elbow_pitch_joint" type="revolute">
     <parent link="elbow_roll_link"/>
@@ -118,8 +234,13 @@
   <!-- ELBOW PITCH LINK -->
   <link name="elbow_pitch_link" >
+    <inertial>
+      <origin xyz="0.0 0 0"  />
+      <mass value="1.0" />
+      <inertia  ixx="1.0" ixy="0.0"  ixz="0.0"  iyy="100.0"  iyz="0.0"  izz="1.0" />
+    </inertial>
     <visual>
       <origin xyz="0.0 0 0" rpy="${M_PI/2} 0 ${M_PI/2+M_PI}" />
       <geometry>
-	<mesh filename="package://clam_description/stl/elbow_pitch_link.STL" scale="${M_SCALE}" />
+        <mesh filename="package://clam_description/stl/elbow_pitch_link.STL" scale="${M_SCALE}" />
       </geometry>
       <material name="Orange" />
@@ -128,8 +249,12 @@
       <origin xyz="0.0 0 0" rpy="${M_PI/2} 0 ${M_PI/2+M_PI}" />
       <geometry>
-	<mesh filename="package://clam_description/stl/elbow_pitch_link_simple.STL" scale="${M_SCALE}" />
+        <mesh filename="package://clam_description/stl/elbow_pitch_link_simple.STL" scale="${M_SCALE}" />
       </geometry>
     </collision>
   </link>
+  <gazebo reference="elbow_pitch_link">
+    <material>Gazebo/Blue</material>
+    <turnGravityOff>false</turnGravityOff>
+  </gazebo>
   <joint name="wrist_roll_joint" type="revolute">
     <parent link="elbow_pitch_link"/>
@@ -142,8 +267,13 @@
   <!-- WRIST ROLL LINK -->
   <link name="wrist_roll_link" >
+    <inertial>
+      <origin xyz="0 0 0"  />
+      <mass value="1.0" />
+      <inertia  ixx="1.0" ixy="0.0"  ixz="0.0"  iyy="100.0"  iyz="0.0"  izz="1.0" />
+    </inertial>
     <visual>
       <origin xyz="0 0 0" rpy="0 ${M_PI/2} ${M_PI/2}" />
       <geometry>
-	<mesh filename="package://clam_description/stl/wrist_roll_link.STL" scale="${M_SCALE}" />
+        <mesh filename="package://clam_description/stl/wrist_roll_link.STL" scale="${M_SCALE}" />
       </geometry>
       <material name="Black" />
@@ -152,8 +282,12 @@
       <origin xyz="0 0 0" rpy="0 ${M_PI/2} ${M_PI/2}" />
       <geometry>
-	<mesh filename="package://clam_description/stl/wrist_roll_link_simple.STL" scale="${M_SCALE}" />
+        <mesh filename="package://clam_description/stl/wrist_roll_link_simple.STL" scale="${M_SCALE}" />
       </geometry>
     </collision>
   </link>
+  <gazebo reference="wrist_roll_link">
+    <material>Gazebo/Blue</material>
+    <turnGravityOff>false</turnGravityOff>
+  </gazebo>
   <joint name="wrist_pitch_joint" type="revolute">
     <parent link="wrist_roll_link"/>
@@ -166,8 +300,13 @@
   <!-- WRIST PITCH LINK -->
   <link name="wrist_pitch_link">
+    <inertial>
+      <origin xyz="0 0 0"  />
+      <mass value="1.0" />
+      <inertia  ixx="1.0" ixy="0.0"  ixz="0.0"  iyy="100.0"  iyz="0.0"  izz="1.0" />
+    </inertial>
     <visual>
       <origin xyz="0 0 0" rpy="${M_PI} -${M_PI/2} 0" />
       <geometry>
-	<mesh filename="package://clam_description/stl/wrist_pitch_link.STL" scale="${M_SCALE}" />
+        <mesh filename="package://clam_description/stl/wrist_pitch_link.STL" scale="${M_SCALE}" />
       </geometry>
       <material name="Grey" />
@@ -176,8 +315,12 @@
       <origin xyz="0 0 0" rpy="${M_PI} -${M_PI/2} 0" />
       <geometry>
-	<mesh filename="package://clam_description/stl/wrist_pitch_link_simple.STL" scale="${M_SCALE}" />
+        <mesh filename="package://clam_description/stl/wrist_pitch_link_simple.STL" scale="${M_SCALE}" />
       </geometry>
     </collision>
   </link>
+  <gazebo reference="wrist_pitch_link">
+    <material>Gazebo/Blue</material>
+    <turnGravityOff>false</turnGravityOff>
+  </gazebo>
   <joint name="gripper_roll_joint" type="revolute">
     <parent link="wrist_pitch_link"/>
@@ -190,12 +333,21 @@
   <!-- GRIPPER ROLL LINK -->
   <link name="gripper_roll_link">
+    <inertial>
+      <origin xyz="0 0 0" />
+      <mass value="1.0" />
+      <inertia  ixx="1.0" ixy="0.0"  ixz="0.0"  iyy="100.0"  iyz="0.0"  izz="1.0" />
+    </inertial>
     <visual>
       <origin xyz="0 0 0" rpy="0 0 0" />
       <geometry>
-	<mesh filename="package://clam_description/stl/gripper_grip_link.STL" scale="1 1 1" />
+        <mesh filename="package://clam_description/stl/gripper_grip_link.STL" scale="1 1 1" />
       </geometry>
       <material name="Orange" />
     </visual>
   </link>
+  <gazebo reference="gripper_roll_link">
+    <material>Gazebo/Blue</material>
+    <turnGravityOff>false</turnGravityOff>
+  </gazebo>
   <joint name="l_gripper_aft_joint" type="revolute">
     <parent link="gripper_roll_link"/>
@@ -203,17 +355,26 @@
     <origin xyz="0.026 .017 0" rpy="${1.04*M_PI} ${M_PI/2} ${34.58*M_PI/180}" />
     <axis xyz="1 0 0" />
-    <limit effort="300" velocity="1" lower="${0*M_PI/180}" upper="${-53*M_PI/180}" />
+    <limit effort="300" velocity="1" lower="${-53*M_PI/180}" upper="${0*M_PI/180}"/>
     <dynamics damping="50" friction="1"/>
   </joint>
   <!-- LEFT GRIPPER AFT LINK -->
   <link name="l_gripper_aft_link">
+    <inertial>
+      <origin xyz="0 0 0"  />
+      <mass value="1.0" />
+      <inertia  ixx="1.0" ixy="0.0"  ixz="0.0"  iyy="100.0"  iyz="0.0"  izz="1.0" />
+    </inertial>
     <visual>
       <origin xyz="0 0 0" rpy="0 0 ${M_PI}" />
       <geometry>
-	<mesh filename="package://clam_description/stl/l_gripper_aft_link.STL" scale="1 1 1" />
-      </geometry>
-      <material name="Grey" />
-    </visual>
-  </link>
+        <mesh filename="package://clam_description/stl/l_gripper_aft_link.STL" scale="1 1 1" />
+      </geometry>
+      <material name="Grey" />
+    </visual>
+  </link>
+  <gazebo reference="l_gripper_aft_link">
+    <material>Gazebo/Blue</material>
+    <turnGravityOff>false</turnGravityOff>
+  </gazebo>
   <joint name="r_gripper_aft_joint" type="revolute">
     <parent link="gripper_roll_link"/>
@@ -227,12 +388,21 @@
   <!-- RIGHT GRIPPER AFT LINK -->
   <link name="r_gripper_aft_link">
+    <inertial>
+      <origin xyz="0 0 0"  />
+      <mass value="1.0" />
+      <inertia  ixx="1.0" ixy="0.0"  ixz="0.0"  iyy="100.0"  iyz="0.0"  izz="1.0" />
+    </inertial>
     <visual>
       <origin xyz="0 0 0" rpy="0 0 ${M_PI}" />
       <geometry>
-	<mesh filename="package://clam_description/stl/r_gripper_aft_link.STL" scale="1 1 1" />
-      </geometry>
-      <material name="Grey" />
-    </visual>
-  </link>
+        <mesh filename="package://clam_description/stl/r_gripper_aft_link.STL" scale="1 1 1" />
+      </geometry>
+      <material name="Grey" />
+    </visual>
+  </link>
+  <gazebo reference="r_gripper_aft_link">
+    <material>Gazebo/Blue</material>
+    <turnGravityOff>false</turnGravityOff>
+  </gazebo>
   <joint name="l_gripper_fwd_joint" type="revolute">
     <parent link="gripper_roll_link"/>
@@ -246,12 +416,21 @@
   <!-- LEFT GRIPPER FWD LINK -->
   <link name="l_gripper_fwd_link">
+    <inertial>
+      <origin xyz="0 0 0"  />
+      <mass value="1.0" />
+      <inertia  ixx="1.0" ixy="0.0"  ixz="0.0"  iyy="100.0"  iyz="0.0"  izz="1.0" />
+    </inertial>
     <visual>
       <origin xyz="0 0 0" rpy="0 0 ${M_PI}" />
       <geometry>
-	<mesh filename="package://clam_description/stl/l_gripper_fwd_link.STL" scale="1 1 1" />
-      </geometry>
-      <material name="Grey" />
-    </visual>
-  </link>
+        <mesh filename="package://clam_description/stl/l_gripper_fwd_link.STL" scale="1 1 1" />
+      </geometry>
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