Commit message: Started creating .sdf version of urdf for gazebo

File: src/clam_description/urdf/clam.urdf (robot description, URDF)
Before this commit: robot clam, 16 links, 15 joints
Links:
- link gripper_fake_tip_link: mass 1.0 -> 0.01
- link tabletop_link: mass 1.0 -> 100.0; geometry collision mesh filename=package://clam_description/stl/tabletop.STL scale=1 1 1; visual mesh filename=package://clam_description/stl/tabletop.STL scale=1 1 1
Joints:
- joint l_gripper_aft_joint: limit lower=0.0 upper=-0.925023722222 effort=300 velocity=1 -> lower=-0.925023722222 upper=0.0 effort=300 velocity=1

File: src/clam_description/urdf/clam.xacro (robot description, xacro)
@@ -22,46 +22,47 @@
   <property name="M_SCALE" value="0.001 0.001 0.001"/>
   <property name="M_PI" value="3.14159"/>
-  <!-- Add a Gazebo plugin controller -->
-  <gazebo>
-    <controller:gazebo_ros_actuator_array
-        name="actuator_array_controller"
-        plugin="libgazebo_ros_actuator_array.so">
-      <alwaysOn>true</alwaysOn>
-      <updateRate>50.0</updateRate>
-      <robotParam>robot_description</robotParam>
-      <joint>
-        <name>joint1</name>
-        <home>0.0</home>
-        <p>10.0</p>
-        <i>0.0</i>
-        <d>0.0</d>
-        <iClamp>0.0</iClamp>
-      </joint>
-      <joint>
-        <name>joint2</name>
-        <home>2.094395102</home>
-        <p>10.0</p>
-        <i>0.0</i>
-        <d>0.0</d>
-        <iClamp>0.0</iClamp>
-      </joint>
-      <joint>
-        <name>joint3</name>
-        <home>1.483529864</home>
-        <p>10.0</p>
-        <i>0.0</i>
-        <d>0.0</d>
-        <iClamp>0.0</iClamp>
-      </joint>
-      <joint>
-        <name>joint4</name>
-        <home>0.0</home>
-        <p>10.0</p>
-        <i>0.0</i>
-        <d>0.0</d>
-        <iClamp>0.0</iClamp>
-      </joint>
-    </controller:gazebo_ros_actuator_array>
-  </gazebo>
+  <!-- Add a Gazebo plugin controller
+       <gazebo>
+       <controller:gazebo_ros_actuator_array
+       name="actuator_array_controller"
+       plugin="libgazebo_ros_actuator_array.so">
+       <alwaysOn>true</alwaysOn>
+       <updateRate>50.0</updateRate>
+       <robotParam>robot_description</robotParam>
+       <joint>
+       <name>joint1</name>
+       <home>0.0</home>
+       <p>10.0</p>
+       <i>0.0</i>
+       <d>0.0</d>
+       <iClamp>0.0</iClamp>
+       </joint>
+       <joint>
+       <name>joint2</name>
+       <home>2.094395102</home>
+       <p>10.0</p>
+       <i>0.0</i>
+       <d>0.0</d>
+       <iClamp>0.0</iClamp>
+       </joint>
+       <joint>
+       <name>joint3</name>
+       <home>1.483529864</home>
+       <p>10.0</p>
+       <i>0.0</i>
+       <d>0.0</d>
+       <iClamp>0.0</iClamp>
+       </joint>
+       <joint>
+       <name>joint4</name>
+       <home>0.0</home>
+       <p>10.0</p>
+       <i>0.0</i>
+       <d>0.0</d>
+       <iClamp>0.0</iClamp>
+       </joint>
+       </controller:gazebo_ros_actuator_array>
+       </gazebo>
+  -->
   <!-- TABLETOP LINK -->
   <joint name="tabletop_joint" type="fixed">
@@ -91,5 +92,5 @@
   </link>
   <gazebo reference="tabletop_link">
-    <material>Gazebo/WoodFloor</material>
+    <material>Gazebo/Blue</material>
     <turnGravityOff>false</turnGravityOff>
   </gazebo>

Commit message: Fixed depreciated warning in dynamixel_hardware_interface

File: src/clam_description/urdf/clam.urdf (robot description, URDF)
Before this commit: robot clam, 16 links, 15 joints
Links:
- link base_link: mass 1.0 -> None

Commit message: Disabled the gripper in the controllers, urdf, etc

File: src/clam_description/urdf/clam.urdf (robot description, URDF)
Before this commit: robot clam, 16 links, 15 joints
Links:
- removed link gripper_fake_tip_link
- removed link l_gripper_aft_link
- removed link l_gripper_fwd_link
- removed link l_gripper_pincher_link
- removed link r_gripper_aft_link
- removed link r_gripper_fwd_link
- removed link r_gripper_pincher_link
Joints:
- removed joint gripper_fake_tip_joint
- removed joint l_gripper_aft_joint
- removed joint l_gripper_aft_pincher_joint
- removed joint l_gripper_fwd_joint
- removed joint r_gripper_aft_joint
- removed joint r_gripper_aft_pincher_joint
- removed joint r_gripper_fwd_joint

Commit message: Solidworks editing

File: src/clam_description/urdf/clam.urdf (robot description, URDF)
Before this commit: robot clam, 9 links, 8 joints
Links:
- link gripper_roll_link: geometry collision mesh filename=package://clam_description/stl/gripper_grip_link_simple.STL scale=1 1 1; visual mesh filename=package://clam_description/stl/gripper_grip_link.STL scale=1 1 1
- link shoulder_pan_link: geometry collision mesh filename=package://clam_description/stl/shoulder_pan_link_simple.STL scale=0.001 0.001 0.001; visual mesh filename=package://clam_description/stl/shoulder_pan_link_simple.STL scale=0.001 0.001 0.001
- link tabletop_link: geometry collision mesh filename=package://clam_description/stl/tabletop_link_simple.STL scale=1 1 1; visual mesh filename=package://clam_description/stl/tabletop.STL scale=1 1 1

File: src/clam_description/urdf/clam.xacro (robot description, xacro)
@@ -84,5 +84,5 @@
       <origin xyz=" 0 0 -0.017"  rpy="${.5*M_PI} 0 ${.5*M_PI}"/>
       <geometry>
-        <mesh filename="package://clam_description/stl/tabletop.STL" scale="1 1 1" />
+        <mesh filename="package://clam_description/stl/tabletop_link_simple.STL" scale="1 1 1" />
       </geometry>
       </collision>>
@@ -141,5 +141,5 @@
       <origin xyz="0 0 0" rpy="0 0 ${M_PI/2}" />
       <geometry>
-        <mesh filename="package://clam_description/stl/shoulder_pan_link.STL" scale="${M_SCALE}" />
+        <mesh filename="package://clam_description/stl/shoulder_pan_link_simple.STL" scale="${M_SCALE}" />
       </geometry>
       <material name="Orange" />

Commit message: Solidworks editing

File: src/clam_description/urdf/clam.urdf (robot description, URDF)
Before this commit: robot clam, 9 links, 8 joints
Links:
- link tabletop_link: geometry collision mesh filename=package://clam_description/stl/tabletop_link_simple.STL scale=0.001 0.001 0.001; visual mesh filename=package://clam_description/stl/tabletop_link_simple.STL scale=0.001 0.001 0.001

File: src/clam_description/urdf/clam.xacro (robot description, xacro)
@@ -77,5 +77,5 @@
       <origin xyz=" 0 0 -0.017"  rpy="${.5*M_PI} 0 ${.5*M_PI}"/>
       <geometry>
-        <mesh filename="package://clam_description/stl/tabletop.STL" scale="1 1 1" />
+        <mesh filename="package://clam_description/stl/tabletop_link_simple.STL" scale="${M_SCALE}" />
       </geometry>
       <material name="Brown" />
@@ -84,5 +84,5 @@
       <origin xyz=" 0 0 -0.017"  rpy="${.5*M_PI} 0 ${.5*M_PI}"/>
       <geometry>
-        <mesh filename="package://clam_description/stl/tabletop_link_simple.STL" scale="1 1 1" />
+        <mesh filename="package://clam_description/stl/tabletop_link_simple.STL" scale="${M_SCALE}" />
       </geometry>
       </collision>>

Commit message: Edited URDF

File: src/clam_description/urdf/clam.urdf (robot description, URDF)
Before this commit: robot clam, 9 links, 8 joints
Links:
- link gripper_roll_link: geometry collision mesh filename=package://clam_description/stl/gripper_grip_link_simple.STL scale=0.001 0.001 0.001; visual mesh filename=package://clam_description/stl/gripper_grip_link.STL scale=0.001 0.001 0.001

File: src/clam_description/urdf/clam.xacro (robot description, xacro)
@@ -339,5 +339,5 @@
       <origin xyz="0 0 0" rpy="0 0 0" />
       <geometry>
-        <mesh filename="package://clam_description/stl/gripper_grip_link.STL" scale="1 1 1" />
+        <mesh filename="package://clam_description/stl/gripper_roll_link.STL" scale="${M_SCALE}" />
       </geometry>
       <material name="Orange" />
@@ -346,5 +346,5 @@
       <origin xyz="0 0 0" rpy="0 0 0" />
       <geometry>
-        <mesh filename="package://clam_description/stl/gripper_grip_link_simple.STL" scale="1 1 1" />
+        <mesh filename="package://clam_description/stl/gripper_roll_link_simple.STL" scale="${M_SCALE}" />
       </geometry>
     </collision>

Commit message: Edited URDF

File: src/clam_description/urdf/clam.urdf (robot description, URDF)
Before this commit: robot clam, 9 links, 8 joints
Links:
- link gripper_roll_link: geometry collision mesh filename=package://clam_description/stl/gripper_roll_link_simple.STL scale=0.001 0.001 0.001; visual mesh filename=package://clam_description/stl/gripper_roll_link.STL scale=0.001 0.001 0.001

Commit message: Tweaking launching procedure

File: src/clam_description/urdf/clam.urdf (robot description, URDF)
Before this commit: robot clam, 9 links, 8 joints
Links:
- link tabletop_link: geometry collision mesh filename=package://clam_description/stl/tabletop_link_simple.STL scale=0.001 0.001 0.001; visual mesh filename=package://clam_description/stl/tabletop_link.STL scale=0.001 0.001 0.001

File: src/clam_description/urdf/clam.xacro (robot description, xacro)
@@ -77,5 +77,5 @@
       <origin xyz=" 0 0 -0.017"  rpy="${.5*M_PI} 0 ${.5*M_PI}"/>
       <geometry>
-        <mesh filename="package://clam_description/stl/tabletop_link_simple.STL" scale="${M_SCALE}" />
+        <mesh filename="package://clam_description/stl/tabletop_link.STL" scale="${M_SCALE}" />
       </geometry>
       <material name="Brown" />

Commit message: Created a dummy fixed gripper

File: src/clam_description/urdf/clam.urdf (robot description, URDF)
Before this commit: robot clam, 9 links, 8 joints
Links:
- added link gripper_finger_link, mass 0.01; collision mesh filename=package://clam_description/stl/gripper_finger_link.STL scale=0.001 0.001 0.001; visual mesh filename=package://clam_description/stl/gripper_finger_link.STL scale=0.001 0.001 0.001
- added link gripper_fixed_finger_link, mass 0.01; collision mesh filename=package://clam_description/stl/gripper_finger_link.STL scale=0.001 0.001 0.001; visual mesh filename=package://clam_description/stl/gripper_finger_link.STL scale=0.001 0.001 0.001
- link gripper_roll_link: geometry collision mesh filename=package://clam_description/stl/gripper_base_link.STL scale=0.001 0.001 0.001; visual mesh filename=package://clam_description/stl/gripper_base_link.STL scale=0.001 0.001 0.001
Joints:
- added joint gripper_finger_joint: type fixed, parent gripper_roll_link, child gripper_finger_link, origin xyz=0.055 -0.0275 0.0 rpy=3.14159 0 0, axis 0 1 0, limit lower=-0.925023722222 upper=0.0 effort=300 velocity=1
- added joint gripper_fixed_finger_joint: type fixed, parent gripper_roll_link, child gripper_fixed_finger_link, origin xyz=0.055 0.0275 0.0 rpy=0 0 0

File: src/clam_description/urdf/clam.xacro (robot description, xacro)
@@ -19,47 +19,4 @@
   <property name="M_SCALE" value="0.001 0.001 0.001"/>
   <property name="M_PI" value="3.14159"/>
-  <!-- Add a Gazebo plugin controller
-       <gazebo>
-       <controller:gazebo_ros_actuator_array
-       name="actuator_array_controller"
-       plugin="libgazebo_ros_actuator_array.so">
-       <alwaysOn>true</alwaysOn>
-       <updateRate>50.0</updateRate>
-       <robotParam>robot_description</robotParam>
-       <joint>
-       <name>joint1</name>
-       <home>0.0</home>
-       <p>10.0</p>
-       <i>0.0</i>
-       <d>0.0</d>
-       <iClamp>0.0</iClamp>
-       </joint>
-       <joint>
-       <name>joint2</name>
-       <home>2.094395102</home>
-       <p>10.0</p>
-       <i>0.0</i>
-       <d>0.0</d>
-       <iClamp>0.0</iClamp>
-       </joint>
-       <joint>
-       <name>joint3</name>
-       <home>1.483529864</home>
-       <p>10.0</p>
-       <i>0.0</i>
-       <d>0.0</d>
-       <iClamp>0.0</iClamp>
-       </joint>
-       <joint>
-       <name>joint4</name>
-       <home>0.0</home>
-       <p>10.0</p>
-       <i>0.0</i>
-       <d>0.0</d>
-       <iClamp>0.0</iClamp>
-       </joint>
-       </controller:gazebo_ros_actuator_array>
-       </gazebo>
-  -->
   <!-- TABLETOP LINK -->
   <joint name="tabletop_joint" type="fixed">
@@ -339,5 +296,5 @@
       <origin xyz="0 0 0" rpy="0 0 0" />
       <geometry>
-        <mesh filename="package://clam_description/stl/gripper_roll_link.STL" scale="${M_SCALE}" />
+        <mesh filename="package://clam_description/stl/gripper_base_link.STL" scale="${M_SCALE}" />
       </geometry>
       <material name="Orange" />
@@ -346,5 +303,5 @@
       <origin xyz="0 0 0" rpy="0 0 0" />
       <geometry>
-        <mesh filename="package://clam_description/stl/gripper_roll_link_simple.STL" scale="${M_SCALE}" />
+        <mesh filename="package://clam_description/stl/gripper_base_link.STL" scale="${M_SCALE}" />
       </geometry>
     </collision>
@@ -354,3 +311,58 @@
     <turnGravityOff>false</turnGravityOff>
   </gazebo>
+  <!-- Gripper Fixed Finger -->
+  <joint name="gripper_fixed_finger_joint" type="fixed">
+    <origin xyz="0.055 0.0275 0.0" rpy="0 0 0" />  <!-- x=up to heaven  y=left to wall z=back towards motor houseing -->
+    <parent link="gripper_roll_link"/>
+    <child link="gripper_fixed_finger_link" />
+  </joint>
+  <link name="gripper_fixed_finger_link" >
+    <inertial>
+      <origin xyz="0 0 0" />
+      <mass value="0.01" />
+      <inertia  ixx="1.0" ixy="0.0"  ixz="0.0"  iyy="100.0"  iyz="0.0"  izz="1.0" />
+    </inertial>
+    <visual>
+      <origin xyz="0 0 0" rpy="0 0 0" />
+      <geometry>
+        <mesh filename="package://clam_description/stl/gripper_finger_link.STL" scale="${M_SCALE}" />
+      </geometry>
+      <material name="Grey" />
+    </visual>
+    <collision>
+      <origin xyz="0 0 0" rpy="0 0 0" />
+      <geometry>
+        <mesh filename="package://clam_description/stl/gripper_finger_link.STL" scale="${M_SCALE}" />
+      </geometry>
+    </collision>
+  </link>
+  <!-- Gripper Moving Finger -->
+  <joint name="gripper_finger_joint" type="fixed">
+    <origin xyz="0.055 -0.0275 0.0" rpy="${M_PI} 0 0" />  <!-- x=up to heaven  y=left to wall z=back towards motor houseing -->
+    <parent link="gripper_roll_link"/>
+    <child link="gripper_finger_link" />
+    <axis xyz="0 1 0" />
+    <limit effort="300" velocity="1" lower="${-53*M_PI/180}" upper="${0*M_PI/180}"/>
+    <dynamics damping="50" friction="1"/>
+  </joint>
+  <link name="gripper_finger_link" >
+    <inertial>
+      <origin xyz="0 0 0" />
+      <mass value="0.01" />
+      <inertia  ixx="1.0" ixy="0.0"  ixz="0.0"  iyy="100.0"  iyz="0.0"  izz="1.0" />
+    </inertial>
+    <visual>
+      <origin xyz="0 0 0" rpy="0 0 0" />
+      <geometry>
+        <mesh filename="package://clam_description/stl/gripper_finger_link.STL" scale="${M_SCALE}" />
+      </geometry>
+      <material name="Grey" />
+    </visual>
+    <collision>
+      <origin xyz="0 0 0" rpy="0 0 0" />
+      <geometry>
+        <mesh filename="package://clam_description/stl/gripper_finger_link.STL" scale="${M_SCALE}" />
+      </geometry>
+    </collision>
+  </link>
 </robot>

Commit message: Transfered new move_group method to clam_block_manipulation package

File: src/clam_description/urdf/clam.urdf (robot description, URDF)
Before this commit: robot clam, 11 links, 10 joints
Links:
- added link gripper_fake_tip_link, mass 0.01; collision sphere radius=.001; visual sphere radius=.001
Joints:
- added joint gripper_fake_tip_joint: type fixed, parent gripper_roll_link, child gripper_fake_tip_link, origin xyz=0.1785 0.0 0.0 rpy=0 0 0

File: src/clam_description/urdf/clam.xacro (robot description, xacro)
@@ -366,3 +366,32 @@
     </collision>
   </link>
+  <!-- FAKE CAMERA CALIBRATION POINT AT GRIPPER TIP -->
+  <joint name="gripper_fake_tip_joint" type="fixed">
+    <origin xyz="0.1785 0.0 0.0" rpy="0 0 0" />
+    <parent link="gripper_roll_link"/>
+    <child link="gripper_fake_tip_link" />
+  </joint>
+  <link name="gripper_fake_tip_link" >
+    <inertial>
+      <origin xyz="0 0 0" />
+      <mass value="0.01" />
+      <inertia  ixx="1.0" ixy="0.0"  ixz="0.0"  iyy="100.0"  iyz="0.0"  izz="1.0" />
+    </inertial>
+    <visual>
+      <origin xyz="0 0 0" rpy="0 0 0" />
+      <geometry>
+        <sphere radius=".001"/>
+      </geometry>
+    </visual>
+    <collision>
+      <origin xyz="-0.1 0 0" rpy="0 0 0" />
+      <geometry>
+        <sphere radius=".001"/>
+      </geometry>
+    </collision>
+  </link>
+  <gazebo reference="gripper_fake_tip_link">
+    <material>Gazebo/Blue</material>
+    <turnGravityOff>false</turnGravityOff>
+  </gazebo>
 </robot>

Commit message: Working on pick service

File: src/clam_description/urdf/clam.urdf (robot description, URDF)
Before this commit: robot clam, 12 links, 11 joints
Links:
- removed link gripper_fake_tip_link
Joints:
- removed joint gripper_fake_tip_joint

File: src/clam_description/urdf/clam.xacro (robot description, xacro)
@@ -367,5 +367,5 @@
   </link>
   <!-- FAKE CAMERA CALIBRATION POINT AT GRIPPER TIP -->
-  <joint name="gripper_fake_tip_joint" type="fixed">
+  <!--joint name="gripper_fake_tip_joint" type="fixed">
     <origin xyz="0.1785 0.0 0.0" rpy="0 0 0" />
     <parent link="gripper_roll_link"/>
@@ -394,4 +394,4 @@
     <material>Gazebo/Blue</material>
     <turnGravityOff>false</turnGravityOff>
-  </gazebo>
+  </gazebo-->
 </robot>

Commit message: Progress on IKFast

File: src/clam_description/urdf/clam.urdf (robot description, URDF)
Before this commit: robot clam, 11 links, 10 joints
Links:
- link shoulder_pan_link: geometry collision mesh filename=package://clam_description/stl/shoulder_pan_link_simple.STL scale=0.001 0.001 0.001; visual mesh filename=package://clam_description/stl/shoulder_pan_link.STL scale=0.001 0.001 0.001
Joints:
- joint elbow_roll_joint: type revolute -> fixed

File: src/clam_description/urdf/clam.xacro (robot description, xacro)
@@ -82,10 +82,4 @@
     <dynamics damping="50" friction="1"/>
   </joint>
-  <transmission name="shoulder_pan_controller" type="pr2_mechanism_model/SimpleTransmission">
-    <actuator name="shoulder_pan_actuator" />
-    <joint name="shoulder_pan_joint" />
-    <mechanicalReduction>1</mechanicalReduction>
-    <motorTorqueConstant>1</motorTorqueConstant>
-  </transmission>
   <!-- SHOULDER PAN LINK -->
   <link name="shoulder_pan_link" >
@@ -98,5 +92,5 @@
       <origin xyz="0 0 0" rpy="0 0 ${M_PI/2}" />
       <geometry>
-        <mesh filename="package://clam_description/stl/shoulder_pan_link_simple.STL" scale="${M_SCALE}" />
+        <mesh filename="package://clam_description/stl/shoulder_pan_link.STL" scale="${M_SCALE}" />
       </geometry>
       <material name="Orange" />
@@ -146,5 +140,5 @@
     <turnGravityOff>false</turnGravityOff>
   </gazebo>
-  <joint name="elbow_roll_joint" type="revolute">
+  <joint name="elbow_roll_joint" type="fixed">
     <parent link="shoulder_pitch_link"/>
     <child link="elbow_roll_link"/>
