Commit message: Working on IKFast stuff

File: src/clam_description/urdf/materials.urdf.xacro (robot description, xacro)
@@ -25,6 +25,3 @@
         <color rgba="1.0 1.0 1.0 1.0"/>
     </material>
-    <material name="GunMetalBrushedAluminum">
-        <texture filename="package://clam_description/media/gun_metal_brushed_aluminum.jpg" />
-    </material>
 </robot>
