Commit message: Created a simplified dae Collada file for IKFast

File: src/clam_description/urdf/clam.7dof.xacro (robot description, xacro)
@@ -82,10 +82,4 @@
     <dynamics damping="50" friction="1"/>
   </joint>
-  <transmission name="shoulder_pan_controller" type="pr2_mechanism_model/SimpleTransmission">
-    <actuator name="shoulder_pan_actuator" />
-    <joint name="shoulder_pan_joint" />
-    <mechanicalReduction>1</mechanicalReduction>
-    <motorTorqueConstant>1</motorTorqueConstant>
-  </transmission>
   <!-- SHOULDER PAN LINK -->
   <link name="shoulder_pan_link" >
@@ -98,5 +92,5 @@
       <origin xyz="0 0 0" rpy="0 0 ${M_PI/2}" />
       <geometry>
-        <mesh filename="package://clam_description/stl/shoulder_pan_link_simple.STL" scale="${M_SCALE}" />
+        <mesh filename="package://clam_description/stl/shoulder_pan_link.STL" scale="${M_SCALE}" />
       </geometry>
       <material name="Orange" />
@@ -367,5 +361,5 @@
   </link>
   <!-- FAKE CAMERA CALIBRATION POINT AT GRIPPER TIP -->
-  <joint name="gripper_fake_tip_joint" type="fixed">
+  <!--joint name="gripper_fake_tip_joint" type="fixed">
     <origin xyz="0.1785 0.0 0.0" rpy="0 0 0" />
     <parent link="gripper_roll_link"/>
@@ -394,4 +388,4 @@
     <material>Gazebo/Blue</material>
     <turnGravityOff>false</turnGravityOff>
-  </gazebo>
+  </gazebo-->
 </robot>
