Commit message: Worked on converage test offset and tolerance

File: src/clam_description/urdf_nogripper/clam.urdf (robot description, URDF)
Before this commit: robot clam, 9 links, 8 joints
Links:
- removed link l_gripper_aft_link
- added link tabletop_link, mass 100.0; collision mesh filename=package://clam_description/stl/tabletop_link_simple.STL scale=0.001 0.001 0.001; visual mesh filename=package://clam_description/stl/tabletop_link.STL scale=0.001 0.001 0.001
- link elbow_pitch_link: mass None -> 1.0
- link elbow_roll_link: mass None -> 1.0
- link gripper_roll_link: mass None -> 1.0; geometry collision mesh filename=package://clam_description/stl/gripper_roll_link_simple.STL scale=0.001 0.001 0.001; visual mesh filename=package://clam_description/stl/gripper_roll_link.STL scale=0.001 0.001 0.001
- link shoulder_pan_link: mass None -> 1.0; geometry collision mesh filename=package://clam_description/stl/shoulder_pan_link_simple.STL scale=0.001 0.001 0.001; visual mesh filename=package://clam_description/stl/shoulder_pan_link_simple.STL scale=0.001 0.001 0.001
- link shoulder_pitch_link: mass None -> 1.0
- link wrist_pitch_link: mass None -> 1.0
- link wrist_roll_link: mass None -> 1.0
Joints:
- removed joint l_gripper_aft_joint
- added joint tabletop_joint: type fixed, parent base_link, child tabletop_link, origin xyz=0 0 0 rpy=0 0 0
