Commit message: Working on OpenRave and Vision

File: src/clam_description/openrave/clam.urdf (robot description, URDF)
Before this commit: robot clam, 9 links, 8 joints
Links:
- removed link elbow_pitch_link
- removed link elbow_roll_link
- removed link gripper_roll_link
- removed link shoulder_pan_link
- removed link shoulder_pitch_link
- removed link tabletop_link
- removed link wrist_pitch_link
- removed link wrist_roll_link
- link base_link: mass 1.0 -> None; geometry visual mesh filename=package://clam_description/openrave/base.stl
Joints:
- removed joint elbow_pitch_joint
- removed joint elbow_roll_joint
- removed joint gripper_roll_joint
- removed joint shoulder_pan_joint
- removed joint shoulder_pitch_joint
- removed joint tabletop_joint
- removed joint wrist_pitch_joint
- removed joint wrist_roll_joint
