Commit message: Added detailed gripper, fixed gripper controller

File: clam_description/urdf/clam.before_gripper_merge.xacro (robot description, xacro)
@@ -305,171 +305,60 @@
     <turnGravityOff>false</turnGravityOff>
   </gazebo>
-  <joint name="gripper_finger_joint" type="revolute">
+  <!-- Gripper Fixed Finger -->
+  <joint name="gripper_fixed_finger_joint" type="fixed">
+    <origin xyz="0.055 0.0275 0.0" rpy="0 0 0" />  <!-- x=up to heaven  y=left to wall z=back towards motor houseing -->
     <parent link="gripper_roll_link"/>
-    <child link="gripper_finger_link"/>
-    <origin xyz="0.026 .017 0" rpy="${1.04*M_PI} ${M_PI/2} ${34.58*M_PI/180}" />
-    <axis xyz="1 0 0" />
+    <child link="gripper_fixed_finger_link" />
+  </joint>
+  <link name="gripper_fixed_finger_link" >
+    <inertial>
+      <origin xyz="0 0 0" />
+      <mass value="0.01" />
+      <inertia  ixx="1.0" ixy="0.0"  ixz="0.0"  iyy="100.0"  iyz="0.0"  izz="1.0" />
+    </inertial>
+    <visual>
+      <origin xyz="0 0 0" rpy="0 0 0" />
+      <geometry>
+        <mesh filename="package://clam_description/stl/gripper_finger_link.STL" scale="${M_SCALE}" />
+      </geometry>
+      <material name="Grey" />
+    </visual>
+    <collision>
+      <origin xyz="0 0 0" rpy="0 0 0" />
+      <geometry>
+        <mesh filename="package://clam_description/stl/gripper_finger_link.STL" scale="${M_SCALE}" />
+      </geometry>
+    </collision>
+  </link>
+  <!-- Gripper Moving Finger -->
+  <joint name="gripper_finger_joint" type="prismatic">
+    <origin xyz="0.055 ${-0.0275 + 0.05} 0.0" rpy="${M_PI} 0 0" />  <!-- x=up to heaven  y=left to wall z=back towards motor housing -->
+    <parent link="gripper_roll_link"/>
+    <child link="gripper_finger_link" />
+    <axis xyz="0 1 0" />
+    <!--limit effort="300" velocity="1" lower="0.05" upper="0"/-->
     <limit effort="300" velocity="1" lower="${-53*M_PI/180}" upper="${0*M_PI/180}"/>
     <dynamics damping="50" friction="1"/>
   </joint>
-  <!-- LEFT GRIPPER AFT LINK -->
-  <link name="gripper_finger_link">
-    <inertial>
-      <origin xyz="0 0 0"  />
-      <mass value="1.0" />
-      <inertia  ixx="1.0" ixy="0.0"  ixz="0.0"  iyy="100.0"  iyz="0.0"  izz="1.0" />
-    </inertial>
-    <visual>
-      <origin xyz="0 0 0" rpy="0 0 ${M_PI}" />
-      <geometry>
-        <mesh filename="package://clam_description/stl/l_gripper_aft_link.STL" scale="1 1 1" />
-      </geometry>
-      <material name="Grey" />
-    </visual>
-  </link>
-  <gazebo reference="l_gripper_aft_link">
-    <material>Gazebo/Blue</material>
-    <turnGravityOff>false</turnGravityOff>
-  </gazebo>
-  <joint name="r_gripper_aft_joint" type="revolute">
-    <parent link="gripper_roll_link"/>
-    <child link="r_gripper_aft_link"/>
-    <origin xyz="0.026 -0.011  0" rpy="${1.345*M_PI} ${M_PI/2} ${34.58*M_PI/180}" />
-    <axis xyz="1 0 0" />
-    <limit effort="300" velocity="1" lower="-3.14" upper="3.14" />
-    <mimic joint="gripper_finger_joint" multiplier="-1.0" offset="0.0" />
-    <dynamics damping="50" friction="1"/>
-  </joint>
-  <!-- RIGHT GRIPPER AFT LINK -->
-  <link name="r_gripper_aft_link">
-    <inertial>
-      <origin xyz="0 0 0"  />
-      <mass value="1.0" />
-      <inertia  ixx="1.0" ixy="0.0"  ixz="0.0"  iyy="100.0"  iyz="0.0"  izz="1.0" />
-    </inertial>
-    <visual>
-      <origin xyz="0 0 0" rpy="0 0 ${M_PI}" />
-      <geometry>
-        <mesh filename="package://clam_description/stl/r_gripper_aft_link.STL" scale="1 1 1" />
-      </geometry>
-      <material name="Grey" />
-    </visual>
-  </link>
-  <gazebo reference="r_gripper_aft_link">
-    <material>Gazebo/Blue</material>
-    <turnGravityOff>false</turnGravityOff>
-  </gazebo>
-  <joint name="l_gripper_fwd_joint" type="revolute">
-    <parent link="gripper_roll_link"/>
-    <child link="l_gripper_fwd_link"/>
-    <origin xyz="0.05 0.008 0.007" rpy="${M_PI*(1+.04)} ${M_PI/2} ${214.58*M_PI/180}" />
-    <axis xyz="1 0 0" />
-    <limit effort="300" velocity="1" lower="0" upper="1.57" />
-    <mimic joint="gripper_finger_joint" multiplier="1.0" offset="0" />
-    <dynamics damping="50" friction="1"/>
-  </joint>
-  <!-- LEFT GRIPPER FWD LINK -->
-  <link name="l_gripper_fwd_link">
-    <inertial>
-      <origin xyz="0 0 0"  />
-      <mass value="1.0" />
-      <inertia  ixx="1.0" ixy="0.0"  ixz="0.0"  iyy="100.0"  iyz="0.0"  izz="1.0" />
-    </inertial>
-    <visual>
-      <origin xyz="0 0 0" rpy="0 0 ${M_PI}" />
-      <geometry>
-        <mesh filename="package://clam_description/stl/l_gripper_fwd_link.STL" scale="1 1 1" />
-      </geometry>
-      <material name="Grey" />
-    </visual>
-  </link>
-  <gazebo reference="l_gripper_fwd_link">
-    <material>Gazebo/Blue</material>
-    <turnGravityOff>false</turnGravityOff>
-  </gazebo>
-  <joint name="r_gripper_fwd_joint" type="revolute">
-    <parent link="gripper_roll_link"/>
-    <child link="r_gripper_fwd_link"/>
-    <origin xyz="0.05 -0.0014 0.007" rpy="${M_PI*(1-.04)} ${M_PI/2} ${145.42*M_PI/180}" />
-    <axis xyz="1 0 0" />
-    <limit effort="300" velocity="1" lower="-1.57" upper="0" />
-    <mimic joint="gripper_finger_joint" multiplier="-1.0" offset="0" />
-    <dynamics damping="50" friction="1"/>
-  </joint>
-  <!-- RIGHT GRIPPER FWD LINK -->
-  <link name="r_gripper_fwd_link">
-    <inertial>
-      <origin xyz="0 0 0"  />
-      <mass value="1.0" />
-      <inertia  ixx="1.0" ixy="0.0"  ixz="0.0"  iyy="100.0"  iyz="0.0"  izz="1.0" />
-    </inertial>
-    <visual>
-      <origin xyz="0 0 0" rpy="0 0 ${M_PI}" />
-      <geometry>
-        <mesh filename="package://clam_description/stl/r_gripper_fwd_link.STL" scale="1 1 1" />
-      </geometry>
-      <material name="Grey" />
-    </visual>
-  </link>
-  <gazebo reference="r_gripper_fwd_link">
-    <material>Gazebo/Blue</material>
-    <turnGravityOff>false</turnGravityOff>
-  </gazebo>
-  <joint name="gripper_finger_pincher_joint" type="continuous">
-    <parent link="gripper_finger_link"/>
-    <child link="l_gripper_pincher_link"/>
-    <origin xyz="-0.0032 0 -0.0508" rpy="${203.27*M_PI/180-.3150*M_PI} 0 0" />
-    <axis xyz="1 0 0" />
-    <limit effort="300" velocity="1" lower="-1.57" upper="1.57" />
-    <mimic joint="gripper_finger_joint" multiplier="-1.0" offset="0" />
-    <dynamics damping="50" friction="1"/>
-  </joint>
-  <!-- LEFT GRIPPER PINCHER -->
-  <link name="l_gripper_pincher_link">
-    <inertial>
-      <origin xyz="0 0 0"  />
-      <mass value="1.0" />
-      <inertia  ixx="1.0" ixy="0.0"  ixz="0.0"  iyy="100.0"  iyz="0.0"  izz="1.0" />
-    </inertial>
-    <visual>
-      <origin xyz="0 0 0" rpy="0 0 ${M_PI}" />
-      <geometry>
-        <mesh filename="package://clam_description/stl/l_gripper_pincher.STL" scale="1 1 1" />
-      </geometry>
-      <material name="Black" />
-    </visual>
-  </link>
-  <gazebo reference="l_gripper_pincher_link">
-    <material>Gazebo/Blue</material>
-    <turnGravityOff>false</turnGravityOff>
-  </gazebo>
-  <joint name="r_gripper_aft_pincher_joint" type="revolute">
-    <parent link="r_gripper_aft_link"/>
-    <child link="r_gripper_pincher_link"/>
-    <origin xyz="0 0 -0.0508" rpy="${23.27*M_PI/180-.3150*M_PI} ${M_PI} 0" />
-    <axis xyz="1 0 0" />
-    <limit effort="300" velocity="1" lower="0" upper="1.57" />
-    <mimic joint="gripper_finger_joint" multiplier="-1.0" offset="0" />
-    <dynamics damping="50" friction="1"/>
-  </joint>
-  <!-- RIGHT GRIPPER PINCHER -->
-  <link name="r_gripper_pincher_link">
-    <inertial>
-      <origin xyz="0 0 0" />
-      <mass value="1.0" />
-      <inertia  ixx="1.0" ixy="0.0"  ixz="0.0"  iyy="100.0"  iyz="0.0"  izz="1.0" />
-    </inertial>
-    <visual>
-      <origin xyz="0 0 0" rpy="0 0 ${M_PI}" />
-      <geometry>
-        <mesh filename="package://clam_description/stl/r_gripper_pincher.STL" scale="1 1 1" />
-      </geometry>
-      <material name="Black" />
-    </visual>
-  </link>
-  <gazebo reference="r_gripper_pincher_link">
-    <material>Gazebo/Blue</material>
-    <turnGravityOff>false</turnGravityOff>
-  </gazebo>
+  <link name="gripper_finger_link" >
+    <inertial>
+      <origin xyz="0 0 0" />
+      <mass value="0.01" />
+      <inertia  ixx="1.0" ixy="0.0"  ixz="0.0"  iyy="100.0"  iyz="0.0"  izz="1.0" />
+    </inertial>
+    <visual>
+      <origin xyz="0 0 0" rpy="0 0 0" />
+      <geometry>
+        <mesh filename="package://clam_description/stl/gripper_finger_link.STL" scale="${M_SCALE}" />
+      </geometry>
+      <material name="Grey" />
+    </visual>
+    <collision>
+      <origin xyz="0 0 0" rpy="0 0 0" />
+      <geometry>
+        <mesh filename="package://clam_description/stl/gripper_finger_link.STL" scale="${M_SCALE}" />
+      </geometry>
+    </collision>
+  </link>
   <!-- FAKE CAMERA CALIBRATION POINT AT GRIPPER TIP -->
   <!--joint name="gripper_fake_tip_joint" type="fixed">

File: clam_description/urdf/clam.urdf (robot description, URDF)
Before this commit: robot clam, 11 links, 10 joints
Links:
- removed link gripper_fixed_finger_link
- added link l_gripper_fwd_link, mass 1.0; visual mesh filename=package://clam_description/stl/l_gripper_fwd_link.STL scale=1 1 1
- added link l_gripper_pincher_link, mass 1.0; visual mesh filename=package://clam_description/stl/l_gripper_pincher.STL scale=1 1 1
- added link r_gripper_aft_link, mass 1.0; visual mesh filename=package://clam_description/stl/r_gripper_aft_link.STL scale=1 1 1
- added link r_gripper_fwd_link, mass 1.0; visual mesh filename=package://clam_description/stl/r_gripper_fwd_link.STL scale=1 1 1
- added link r_gripper_pincher_link, mass 1.0; visual mesh filename=package://clam_description/stl/r_gripper_pincher.STL scale=1 1 1
- link gripper_finger_link: mass 0.01 -> 1.0; geometry visual mesh filename=package://clam_description/stl/l_gripper_aft_link.STL scale=1 1 1
Joints:
- removed joint gripper_fixed_finger_joint
- added joint gripper_finger_pincher_joint: type continuous, parent gripper_finger_link, child l_gripper_pincher_link, origin xyz=-0.0032 0 -0.0508 rpy=2.55812692389 0 0, axis 1 0 0, limit lower=-1.57 upper=1.57 effort=300 velocity=1, mimic joint=gripper_finger_joint multiplier=-1.0 offset=0
- added joint l_gripper_fwd_joint: type revolute, parent gripper_roll_link, child l_gripper_fwd_link, origin xyz=0.05 0.008 0.007 rpy=3.2672536 1.570795 3.74512434556, axis 1 0 0, limit lower=0 upper=1.57 effort=300 velocity=1, mimic joint=gripper_finger_joint multiplier=1.0 offset=0
- added joint r_gripper_aft_joint: type revolute, parent gripper_roll_link, child r_gripper_aft_link, origin xyz=0.026 -0.011  0 rpy=4.22543855 1.570795 0.603534345556, axis 1 0 0, limit lower=-3.14 upper=3.14 effort=300 velocity=1, mimic joint=gripper_finger_joint multiplier=-1.0 offset=0.0
- added joint r_gripper_aft_pincher_joint: type revolute, parent r_gripper_aft_link, child r_gripper_pincher_link, origin xyz=0 0 -0.0508 rpy=-0.583463076111 3.14159 0, axis 1 0 0, limit lower=0 upper=1.57 effort=300 velocity=1, mimic joint=gripper_finger_joint multiplier=-1.0 offset=0
- added joint r_gripper_fwd_joint: type revolute, parent gripper_roll_link, child r_gripper_fwd_link, origin xyz=0.05 -0.0014 0.007 rpy=3.0159264 1.570795 2.53805565444, axis 1 0 0, limit lower=-1.57 upper=0 effort=300 velocity=1, mimic joint=gripper_finger_joint multiplier=-1.0 offset=0
- joint gripper_finger_joint: axis 0 1 0 -> 1 0 0; limit lower=0.05 upper=0 effort=300 velocity=1 -> lower=-0.925023722222 upper=0.0 effort=300 velocity=1; origin xyz=0.055 0.0225 0.0 rpy=3.14159 0 0 -> xyz=0.026 .017 0 rpy=3.2672536 1.570795 0.603534345556; type prismatic -> revolute
