Commit message: Put ClamArm in Gazebo, Renamed ikfast plugin

File: clam_description/urdf/clam.xacro (robot description, xacro)
@@ -2,18 +2,14 @@
 <!-- Robot Description format of CLAM arm
 Dave Coleman - davetcoleman@gmail.com
-12/20/2012
+10/23/13
 Documentation:
 URDF
 http://www.ros.org/wiki/urdf/XML
-Joint Safety Limits
-http://www.ros.org/wiki/pr2_controller_manager/safety_limits
 XARCO - Macro Language
 http://www.ros.org/wiki/xacro
-Gazebo Modeling
-http://www.ros.org/wiki/simulator_gazebo/Tutorials/SpawningObjectInSimulation
 -->
-<robot name="clam">
+<robot name="clam" xmlns:xacro="http://www.ros.org/wiki/xacro">
   <!-- Include materials -->
-  <include filename="$(find clam_description)/urdf/materials.urdf.xacro" />
+  <xacro:include filename="$(find clam_description)/urdf/materials.urdf.xacro" />
   <!-- Constants -->
   <property name="M_SCALE" value="0.001 0.001 0.001"/>
@@ -46,6 +42,5 @@
   </link>
   <gazebo reference="tabletop_link">
-    <material>Gazebo/Blue</material>
-    <turnGravityOff>false</turnGravityOff>
+    <material>Gazebo/White</material>
   </gazebo>
   <!-- BASE LINK -->
@@ -71,6 +66,5 @@
   </link>
   <gazebo reference="base_link">
-    <material>Gazebo/Blue</material>
-    <turnGravityOff>false</turnGravityOff>
+    <material>Gazebo/Grey</material>
   </gazebo>
   <joint name="shoulder_pan_joint" type="revolute">
@@ -104,6 +98,5 @@
   </link>
   <gazebo reference="shoulder_pan_link">
-    <material>Gazebo/Blue</material>
-    <turnGravityOff>false</turnGravityOff>
+    <material>Gazebo/Orange</material>
   </gazebo>
   <joint name="shoulder_pitch_joint" type="revolute">
@@ -137,6 +130,5 @@
   </link>
   <gazebo reference="shoulder_pitch_link">
-    <material>Gazebo/Blue</material>
-    <turnGravityOff>false</turnGravityOff>
+    <material>Gazebo/Grey</material>
   </gazebo>
   <joint name="elbow_roll_joint" type="revolute">
@@ -170,6 +162,5 @@
   </link>
   <gazebo reference="elbow_roll_link">
-    <material>Gazebo/Blue</material>
-    <turnGravityOff>false</turnGravityOff>
+    <material>Gazebo/Black</material>
   </gazebo>
   <joint name="elbow_pitch_joint" type="revolute">
@@ -203,6 +194,5 @@
   </link>
   <gazebo reference="elbow_pitch_link">
-    <material>Gazebo/Blue</material>
-    <turnGravityOff>false</turnGravityOff>
+    <material>Gazebo/Orange</material>
   </gazebo>
   <joint name="wrist_roll_joint" type="revolute">
@@ -236,6 +226,5 @@
   </link>
   <gazebo reference="wrist_roll_link">
-    <material>Gazebo/Blue</material>
-    <turnGravityOff>false</turnGravityOff>
+    <material>Gazebo/Black</material>
   </gazebo>
   <joint name="wrist_pitch_joint" type="revolute">
@@ -269,6 +258,5 @@
   </link>
   <gazebo reference="wrist_pitch_link">
-    <material>Gazebo/Blue</material>
-    <turnGravityOff>false</turnGravityOff>
+    <material>Gazebo/Grey</material>
   </gazebo>
   <joint name="gripper_roll_joint" type="revolute">
@@ -302,6 +290,5 @@
   </link>
   <gazebo reference="gripper_roll_link">
-    <material>Gazebo/Blue</material>
-    <turnGravityOff>false</turnGravityOff>
+    <material>Gazebo/Orange</material>
   </gazebo>
   <joint name="gripper_finger_joint" type="revolute">
@@ -329,6 +316,5 @@
   </link>
   <gazebo reference="l_gripper_aft_link">
-    <material>Gazebo/Blue</material>
-    <turnGravityOff>false</turnGravityOff>
+    <material>Gazebo/Grey</material>
   </gazebo>
   <joint name="r_gripper_aft_joint" type="revolute">
@@ -357,6 +343,5 @@
   </link>
   <gazebo reference="r_gripper_aft_link">
-    <material>Gazebo/Blue</material>
-    <turnGravityOff>false</turnGravityOff>
+    <material>Gazebo/Grey</material>
   </gazebo>
   <joint name="l_gripper_fwd_joint" type="revolute">
@@ -385,6 +370,5 @@
   </link>
   <gazebo reference="l_gripper_fwd_link">
-    <material>Gazebo/Blue</material>
-    <turnGravityOff>false</turnGravityOff>
+    <material>Gazebo/Grey</material>
   </gazebo>
   <joint name="r_gripper_fwd_joint" type="revolute">
@@ -413,6 +397,5 @@
   </link>
   <gazebo reference="r_gripper_fwd_link">
-    <material>Gazebo/Blue</material>
-    <turnGravityOff>false</turnGravityOff>
+    <material>Gazebo/Grey</material>
   </gazebo>
   <joint name="gripper_finger_pincher_joint" type="revolute">
@@ -441,6 +424,5 @@
   </link>
   <gazebo reference="l_gripper_pincher_link">
-    <material>Gazebo/Blue</material>
-    <turnGravityOff>false</turnGravityOff>
+    <material>Gazebo/Black</material>
   </gazebo>
   <joint name="r_gripper_aft_pincher_joint" type="revolute">
@@ -469,6 +451,76 @@
   </link>
   <gazebo reference="r_gripper_pincher_link">
-    <material>Gazebo/Blue</material>
-    <turnGravityOff>false</turnGravityOff>
+    <material>Gazebo/Black</material>
+  </gazebo>
+  <!-- Transmissions for ROS Control -->
+  <transmission name="tran1">
+    <type>transmission_interface/SimpleTransmission</type>
+    <joint name="shoulder_pan_joint"/>
+    <actuator name="motor1">
+      <hardwareInterface>EffortJointInterface</hardwareInterface>
+      <mechanicalReduction>1</mechanicalReduction>
+    </actuator>
+  </transmission>
+  <transmission name="tran1">
+    <type>transmission_interface/SimpleTransmission</type>
+    <joint name="shoulder_pitch_joint"/>
+    <actuator name="motor1">
+      <hardwareInterface>EffortJointInterface</hardwareInterface>
+      <mechanicalReduction>1</mechanicalReduction>
+    </actuator>
+  </transmission>
+  <transmission name="tran1">
+    <type>transmission_interface/SimpleTransmission</type>
+    <joint name="elbow_roll_joint"/>
+    <actuator name="motor1">
+      <hardwareInterface>EffortJointInterface</hardwareInterface>
+      <mechanicalReduction>1</mechanicalReduction>
+    </actuator>
+  </transmission>
+  <transmission name="tran1">
+    <type>transmission_interface/SimpleTransmission</type>
+    <joint name="elbow_pitch_joint"/>
+    <actuator name="motor1">
+      <hardwareInterface>EffortJointInterface</hardwareInterface>
+      <mechanicalReduction>1</mechanicalReduction>
+    </actuator>
+  </transmission>
+  <transmission name="tran1">
+    <type>transmission_interface/SimpleTransmission</type>
+    <joint name="wrist_roll_joint"/>
+    <actuator name="motor1">
+      <hardwareInterface>EffortJointInterface</hardwareInterface>
+      <mechanicalReduction>1</mechanicalReduction>
+    </actuator>
+  </transmission>
+  <transmission name="tran1">
+    <type>transmission_interface/SimpleTransmission</type>
+    <joint name="wrist_pitch_joint"/>
+    <actuator name="motor1">
+      <hardwareInterface>EffortJointInterface</hardwareInterface>
+      <mechanicalReduction>1</mechanicalReduction>
+    </actuator>
+  </transmission>
+  <transmission name="tran1">
+    <type>transmission_interface/SimpleTransmission</type>
+    <joint name="gripper_roll_joint"/>
+    <actuator name="motor1">
+      <hardwareInterface>EffortJointInterface</hardwareInterface>
+      <mechanicalReduction>1</mechanicalReduction>
+    </actuator>
+  </transmission>
+  <transmission name="tran1">
+    <type>transmission_interface/SimpleTransmission</type>
+    <joint name="gripper_finger_joint"/>
+    <actuator name="motor1">
+      <hardwareInterface>EffortJointInterface</hardwareInterface>
+      <mechanicalReduction>1</mechanicalReduction>
+    </actuator>
+  </transmission>
+  <!-- ros_control plugin -->
+  <gazebo>
+    <plugin name="gazebo_ros_control" filename="libgazebo_ros_control.so">
+      <robotNamespace>/clam</robotNamespace>
+    </plugin>
   </gazebo>
   <!-- FAKE CAMERA CALIBRATION POINT AT GRIPPER TIP -->
@@ -498,6 +550,5 @@
   </link>
   <gazebo reference="gripper_fake_tip_link">
-    <material>Gazebo/Blue</material>
-    <turnGravityOff>false</turnGravityOff>
+    <material>Gazebo/Grey</material>
   </gazebo-->
 </robot>
