Commit message: Enabled 7th dof, worked on caching ik results

File: clam_description/urdf/clam.urdf (robot description, URDF)
Before this commit: robot clam, 11 links, 10 joints
Joints:
- joint elbow_roll_joint: type fixed -> revolute

File: clam_description/urdf/clam.xacro (robot description, xacro)
@@ -140,5 +140,5 @@
     <turnGravityOff>false</turnGravityOff>
   </gazebo>
-  <joint name="elbow_roll_joint" type="fixed">
+  <joint name="elbow_roll_joint" type="revolute">
     <parent link="shoulder_pitch_link"/>
     <child link="elbow_roll_link"/>

Commit message: Working on IKFast

File: clam_description/urdf/clam.urdf (robot description, URDF)
Before this commit: robot clam, 11 links, 10 joints
Links:
- removed link tabletop_link
Joints:
- removed joint tabletop_joint
- joint elbow_roll_joint: type revolute -> fixed

File: clam_description/urdf/clam.xacro (robot description, xacro)
@@ -20,5 +20,5 @@
   <property name="M_PI" value="3.14159"/>
   <!-- TABLETOP LINK -->
-  <joint name="tabletop_joint" type="fixed">
+  <!--joint name="tabletop_joint" type="fixed">
     <origin xyz="0 0 0" rpy="0 0 0" />
     <parent link="base_link"/>
@@ -48,5 +48,5 @@
     <material>Gazebo/Blue</material>
     <turnGravityOff>false</turnGravityOff>
-  </gazebo>
+  </gazebo-->
   <!-- BASE LINK -->
   <link name="base_link">
@@ -140,5 +140,5 @@
     <turnGravityOff>false</turnGravityOff>
   </gazebo>
-  <joint name="elbow_roll_joint" type="revolute">
+  <joint name="elbow_roll_joint" type="fixed">
     <parent link="shoulder_pitch_link"/>
     <child link="elbow_roll_link"/>

Commit message: Updated for MoveIt API changes

File: clam_description/urdf/clam.urdf (robot description, URDF)
Before this commit: robot clam, 10 links, 9 joints
Links:
- added link tabletop_link, mass 100.0; collision mesh filename=package://clam_description/stl/tabletop_link_simple.STL scale=0.001 0.001 0.001; visual mesh filename=package://clam_description/stl/tabletop_link.STL scale=0.001 0.001 0.001
Joints:
- added joint tabletop_joint: type fixed, parent base_link, child tabletop_link, origin xyz=0 0 0 rpy=0 0 0

File: clam_description/urdf/clam.xacro (robot description, xacro)
@@ -20,5 +20,5 @@
   <property name="M_PI" value="3.14159"/>
   <!-- TABLETOP LINK -->
-  <!--joint name="tabletop_joint" type="fixed">
+  <joint name="tabletop_joint" type="fixed">
     <origin xyz="0 0 0" rpy="0 0 0" />
     <parent link="base_link"/>
@@ -48,5 +48,5 @@
     <material>Gazebo/Blue</material>
     <turnGravityOff>false</turnGravityOff>
-  </gazebo-->
+  </gazebo>
   <!-- BASE LINK -->
   <link name="base_link">

Commit message: Got gripper controller to work in simulation

File: clam_description/urdf/clam.urdf (robot description, URDF)
Before this commit: robot clam, 11 links, 10 joints
Joints:
- joint gripper_finger_joint: limit lower=-0.925023722222 upper=0.0 effort=300 velocity=1 -> lower=0.05 upper=0 effort=300 velocity=1; origin xyz=0.055 -0.0275 0.0 rpy=3.14159 0 0 -> xyz=0.055 0.0225 0.0 rpy=3.14159 0 0; type fixed -> prismatic

File: clam_description/urdf/clam.xacro (robot description, xacro)
@@ -332,10 +332,10 @@
   </link>
   <!-- Gripper Moving Finger -->
-  <joint name="gripper_finger_joint" type="fixed">
-    <origin xyz="0.055 -0.0275 0.0" rpy="${M_PI} 0 0" />  <!-- x=up to heaven  y=left to wall z=back towards motor houseing -->
+  <joint name="gripper_finger_joint" type="prismatic">
+    <origin xyz="0.055 ${-0.0275 + 0.05} 0.0" rpy="${M_PI} 0 0" />  <!-- x=up to heaven  y=left to wall z=back towards motor houseing -->
     <parent link="gripper_roll_link"/>
     <child link="gripper_finger_link" />
     <axis xyz="0 1 0" />
-    <limit effort="300" velocity="1" lower="${-53*M_PI/180}" upper="${0*M_PI/180}"/>
+    <limit effort="300" velocity="1" lower="0.05" upper="0"/>
     <dynamics damping="50" friction="1"/>
   </joint>

Commit message: Updated urdf

File: clam_description/urdf/clam.urdf (robot description, URDF)
Before this commit: robot clam, 15 links, 14 joints
Joints:
- joint gripper_finger_pincher_joint: mimic joint=gripper_finger_joint multiplier=-1.0 offset=0 -> joint=gripper_finger_joint multiplier=-1.0 offset=0.0; type continuous -> revolute
- joint l_gripper_fwd_joint: mimic joint=gripper_finger_joint multiplier=1.0 offset=0 -> joint=gripper_finger_joint multiplier=1.0 offset=0.0
- joint r_gripper_aft_pincher_joint: mimic joint=gripper_finger_joint multiplier=-1.0 offset=0 -> joint=gripper_finger_joint multiplier=-1.0 offset=0.0
- joint r_gripper_fwd_joint: mimic joint=gripper_finger_joint multiplier=-1.0 offset=0 -> joint=gripper_finger_joint multiplier=-1.0 offset=0.0

File: clam_description/urdf/clam.xacro (robot description, xacro)
@@ -366,5 +366,5 @@
     <axis xyz="1 0 0" />
     <limit effort="300" velocity="1" lower="0" upper="1.57" />
-    <mimic joint="gripper_finger_joint" multiplier="1.0" offset="0" />
+    <mimic joint="gripper_finger_joint" multiplier="1.0" offset="0.0" />
     <dynamics damping="50" friction="1"/>
   </joint>
@@ -394,5 +394,5 @@
     <axis xyz="1 0 0" />
     <limit effort="300" velocity="1" lower="-1.57" upper="0" />
-    <mimic joint="gripper_finger_joint" multiplier="-1.0" offset="0" />
+    <mimic joint="gripper_finger_joint" multiplier="-1.0" offset="0.0" />
     <dynamics damping="50" friction="1"/>
   </joint>
@@ -416,5 +416,5 @@
     <turnGravityOff>false</turnGravityOff>
   </gazebo>
-  <joint name="gripper_finger_pincher_joint" type="continuous">
+  <joint name="gripper_finger_pincher_joint" type="revolute">
     <parent link="gripper_finger_link"/>
     <child link="l_gripper_pincher_link"/>
@@ -422,5 +422,5 @@
     <axis xyz="1 0 0" />
     <limit effort="300" velocity="1" lower="-1.57" upper="1.57" />
-    <mimic joint="gripper_finger_joint" multiplier="-1.0" offset="0" />
+    <mimic joint="gripper_finger_joint" multiplier="-1.0" offset="0.0" />
     <dynamics damping="50" friction="1"/>
   </joint>
@@ -450,5 +450,5 @@
     <axis xyz="1 0 0" />
     <limit effort="300" velocity="1" lower="0" upper="1.57" />
-    <mimic joint="gripper_finger_joint" multiplier="-1.0" offset="0" />
+    <mimic joint="gripper_finger_joint" multiplier="-1.0" offset="0.0" />
     <dynamics damping="50" friction="1"/>
   </joint>

Commit message: Mimic tag and full gripper support

File: clam_description/urdf/clam.urdf (robot description, URDF)
Before this commit: robot clam, 15 links, 14 joints
Links:
- link gripper_roll_link: geometry collision mesh filename=package://clam_description/stl/gripper_roll_link.STL scale=0.001 0.001 0.001; visual mesh filename=package://clam_description/stl/gripper_roll_link.STL scale=0.001 0.001 0.001

File: clam_description/urdf/clam.xacro (robot description, xacro)
@@ -290,5 +290,5 @@
       <origin xyz="0 0 0" rpy="0 0 0" />
       <geometry>
-        <mesh filename="package://clam_description/stl/gripper_base_link.STL" scale="${M_SCALE}" />
+        <mesh filename="package://clam_description/stl/gripper_roll_link.STL" scale="${M_SCALE}" />
       </geometry>
       <material name="Orange" />
@@ -297,5 +297,5 @@
       <origin xyz="0 0 0" rpy="0 0 0" />
       <geometry>
-        <mesh filename="package://clam_description/stl/gripper_base_link.STL" scale="${M_SCALE}" />
+        <mesh filename="package://clam_description/stl/gripper_roll_link.STL" scale="${M_SCALE}" />
       </geometry>
     </collision>

Commit message: Created new method for doing pick place, borrowed from Baxter

File: clam_description/urdf/clam.urdf (robot description, URDF)
Before this commit: robot clam, 15 links, 14 joints
Links:
- removed link tabletop_link
Joints:
- removed joint tabletop_joint
